File: amiga crossover.kicad_pcb (KiCad board)
At the start: 2 copper layers, 119.9 x 114.2 mm, 19 parts, among them M3 MountingHole_3.2mm_M3

Commit message: updated readme
Other:
- board text added: "Line In"
- board text added: "Tweeter Out"
- board text removed: "Tweet Out"
Changed lines of the file:
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@@
   (general
     (thickness 1.6)
-    (drawings 7)
+    (drawings 8)
     (tracks 66)
     (zones 0)
@@
     )
   )
+  (gr_text "Line In" (at 110.49 88.9) (layer F.SilkS)
+    (effects (font (size 2 2) (thickness 0.15)))
+  )
   (gr_line (start 102.616 21.209) (end 102.616 135.382) (layer Edge.Cuts) (width 0.05))
   (gr_line (start 222.504 21.209) (end 102.616 21.209) (layer Edge.Cuts) (width 0.05))
   (gr_line (start 222.504 135.382) (end 222.504 21.209) (layer Edge.Cuts) (width 0.05))
   (gr_line (start 102.616 135.382) (end 222.504 135.382) (layer Edge.Cuts) (width 0.05))
-  (gr_text "Amiga Crossover Oct 2019 - laxprad.ca" (at 220.091 67.564 90) (layer F.SilkS)
+  (gr_text "Amiga Crossover Oct 2019 - laxprad.ca" (at 219.71 46.99 90) (layer F.SilkS)
     (effects (font (size 1.5 1.5) (thickness 0.3)))
   )
-  (gr_text "Tweet Out" (at 206.756 45.72) (layer F.SilkS)
+  (gr_text "Tweeter Out" (at 208.28 45.72) (layer F.SilkS)
     (effects (font (size 2 2) (thickness 0.15)))
   )
